Commit message: Remove transmissions

File: ars_description/urdf/parts/chassis.xacro (robot description, xacro)
@@ -2,5 +2,6 @@
 <robot xmlns:xacro="http://www.ros.org/wiki/xacro">
     <xacro:macro name="chassis">
-        <link name="${base_link_name}">
+        <link name="base_link"/>
+        <link name="chassis">
             <collision>
                 <origin xyz="0 0 0" rpy="0 0 0"/>
@@ -18,13 +19,4 @@
                 </material>
             </visual>
-        </link>
-        <!-- Fixed joint to add dummy inertia link -->
-        <joint name="base_to_base_inertia" type="fixed">
-            <parent link="${base_link_name}"/>
-            <child link="base_inertia"/>
-            <origin xyz="0 0 0" rpy="0 0 0"/>
-        </joint>
-        <!-- Dummy inertia link, because KDL cannot have inertia on the base link -->
-        <link name="base_inertia">
             <inertial>
                 <origin xyz="0 0 0" rpy="0 0 0"/>
@@ -38,4 +30,10 @@
             </inertial>
         </link>
+        <!-- Fixed joint to add dummy inertia link -->
+        <joint name="chassis_joinz" type="fixed">
+            <parent link="base_link"/>
+            <child link="chassis"/>
+            <origin xyz="0 0 0" rpy="0 0 0"/>
+        </joint>
     </xacro:macro>
 </robot>
