Commit message: Changed wheel collision model to sphere

File: ars_description/urdf/parts/front_wheel.xacro (robot description, xacro)
@@ -13,5 +13,5 @@
                 <origin xyz="0 0 0" rpy="0 0 0" />
                 <geometry>
-                    <cylinder length="${wheelWidth}" radius="${wheelRadius}"/>
+                    <sphere radius="${wheelRadius}"/>
                 </geometry>
             </collision>

File: ars_description/urdf/parts/rear_wheel.xacro (robot description, xacro)
@@ -12,5 +12,5 @@
                 <origin xyz="0 0 0" rpy="0 0 0" />
                 <geometry>
-                    <cylinder length="${wheelWidth}" radius="${wheelRadius}"/>
+                    <sphere radius="${wheelRadius}"/>
                 </geometry>
             </collision>
