Commit message: Save progress

File: ars_description/urdf/parts/hinge.xacro (robot description, xacro)
@@ -6,5 +6,5 @@
             <child link="${prefix}_HINGE"/>
             <origin xyz="${X} ${Y} ${wheelHeight - chassisHeight/2.0}" rpy="-${0.5*PI} 0.0 0.0"/>
-            <axis xyz="0 -1 0" rpy="0 0 0"/>
+            <axis xyz="0 1 0" rpy="0 0 0"/>
         </joint>
         <link name="${prefix}_HINGE">

File: ars_description/urdf/parts/rear_wheel.xacro (robot description, xacro)
@@ -7,4 +7,5 @@
             <origin xyz="${X} ${Y} ${wheelHeight - chassisHeight/2.0}" rpy="${PI/2} 0 0" />
             <axis xyz="0 0 -1" rpy="0 0 0" />
+            <dynamics damping="0.2" />
         </joint>
         <link name="${prefix}_REAR_WHEEL">

File: ars_description/urdf/ros2_control.xacro (robot description, xacro)
@@ -29,5 +29,5 @@
             <ros>
                 <namespace></namespace>
-                <remapping>ackermann_steering_controller/reference_:=cmd_vel_stamped</remapping>
+                <remapping>ackermann_steering_controller/reference_:=cmd_vel</remapping>
                 <remapping>ackermann_steering_controller/odometry:=odom</remapping>
                 <remapping>ackermann_steering_controller/tf_odometry:=tf</remapping>
