Commit message: Adding Gazebo plugins and Transmissions

File: ars_description/urdf/arc.xacro (robot description, xacro)
@@ -10,4 +10,6 @@
     <xacro:include filename="$(find ars_description)/urdf/sensors/imu.xacro"/>
     <xacro:include filename="$(find ars_description)/urdf/sensors/lidar.xacro"/>
+    <xacro:include filename="$(find ars_description)/urdf/arc.gazebo"/>
+    <xacro:include filename="$(find ars_description)/urdf/arc_transmissions.xacro"/>
     <xacro:chassis/>
     <xacro:hinge prefix="LEFT"

File: ars_description/urdf/properties.xacro (robot description, xacro)
@@ -1,6 +1,8 @@
 <?xml version="1.0"?>
 <robot xmlns:xacro="http://www.ros.org/wiki/xacro">
+    <xacro:property name="base_link_name" value="base_link"/>
     <xacro:property name="PI" value="3.1415926535897931"/>
-    <xacro:property name="base_link_name" value="base_link"/>
+    <xacro:property name="friction_coeff" value="0.8"/>
+    <xacro:property name="transmission_reduction" value="1"/>
     <!-- Chassis properties -->
     <xacro:property name="chassisHeight" value="0.075"/>

Commit message: ros2_control

File: ars_description/urdf/arc.xacro (robot description, xacro)
@@ -10,6 +10,6 @@
     <xacro:include filename="$(find ars_description)/urdf/sensors/imu.xacro"/>
     <xacro:include filename="$(find ars_description)/urdf/sensors/lidar.xacro"/>
-    <xacro:include filename="$(find ars_description)/urdf/arc.gazebo"/>
-    <xacro:include filename="$(find ars_description)/urdf/arc_transmissions.xacro"/>
+    <xacro:include filename="$(find ars_description)/urdf/gazebo.xacro"/>
+    <xacro:include filename="$(find ars_description)/urdf/transmissions.xacro"/>
     <xacro:chassis/>
     <xacro:hinge prefix="LEFT"
@@ -21,18 +21,14 @@
     <xacro:front_wheel prefix="LEFT"
         X="0"
-        Y="${hingeLength/2+wheelWidth/2}"
-        friction_coeff="0.5"/>
+        Y="${hingeLength/2+wheelWidth/2}"/>
     <xacro:front_wheel prefix="RIGHT"
         X="0"
-        Y="${-hingeLength/2-wheelWidth/2}"
-        friction_coeff="0.5"/>
+        Y="${-hingeLength/2-wheelWidth/2}"/>
     <xacro:rear_wheel prefix="LEFT"
         X="${backWheelX}"
-        Y="${chassisWidth/2+wheelClearance+wheelWidth/2}"
-        friction_coeff="0.0"/>
+        Y="${chassisWidth/2+wheelClearance+wheelWidth/2}"/>
     <xacro:rear_wheel prefix="RIGHT"
         X="${backWheelX}"
-        Y="${-chassisWidth/2-wheelClearance-wheelWidth/2}"
-        friction_coeff="0.0"/>
+        Y="${-chassisWidth/2-wheelClearance-wheelWidth/2}"/>
     <xacro:IMU base_link="${base_link_name}"/>
     <xacro:LIDAR base_link="${base_link_name}"/>

File: ars_description/urdf/gazebo.xacro (robot description, xacro)
@@ -1,4 +1,64 @@
 <?xml version="1.0" ?>
-<robot>
+<robot xmlns:xacro="http://www.ros.org/wiki/xacro">
+    <ros2_control name="IgnitionSystem" type="system">
+        <hardware>
+            <plugin>ign_ros2_control/IgnitionSystem</plugin>
+        </hardware>
+        <joint name="LEFT_FRONT_WHEEL_JOINT">
+            <command_interface name="velocity">
+                <param name="min">-1000</param>
+                <param name="max">1000</param>
+            </command_interface>
+            <state_interface name="position"/>
+            <state_interface name="velocity"/>
+        </joint>
+        <joint name="RIGHT_FRONT_WHEEL_JOINT">
+            <command_interface name="velocity">
+                <param name="min">-1000</param>
+                <param name="max">1000</param>
+            </command_interface>
+            <state_interface name="position"/>
+            <state_interface name="velocity"/>
+        </joint>
+        <joint name="LEFT_HINGE_JOINT">
+            <command_interface name="velocity">
+                <param name="min">-1000</param>
+                <param name="max">1000</param>
+            </command_interface>
+            <state_interface name="position"/>
+            <state_interface name="velocity"/>
+        </joint>
+        <joint name="RIGHT_HINGE_JOINT">
+            <command_interface name="velocity">
+                <param name="min">-1000</param>
+                <param name="max">1000</param>
+            </command_interface>
+            <state_interface name="position"/>
+            <state_interface name="velocity"/>
+        </joint>
+        <joint name="LEFT_REAR_WHEEL_JOINT">
+            <command_interface name="velocity">
+                <param name="min">-1000</param>
+                <param name="max">1000</param>
+            </command_interface>
+            <state_interface name="position"/>
+            <state_interface name="velocity"/>
+        </joint>
+        <joint name="RIGHT_REAR_WHEEL_JOINT">
+            <command_interface name="velocity">
+                <param name="min">-1000</param>
+                <param name="max">1000</param>
+            </command_interface>
+            <state_interface name="position"/>
+            <state_interface name="velocity"/>
+        </joint>
+    </ros2_control>
+    <gazebo>
+        <!-- Joint state publisher -->
+        <plugin filename="ign_ros2_control-system" name="ign_ros2_control::IgnitionROS2ControlPlugin">
+            <parameters>$(find ars_description)/config/ars_description.yaml</parameters>
+        </plugin>
+    </gazebo>
+    <!--        Sensors        -->
     <!-- IMU -->
     <gazebo reference="imu_link">
@@ -47,5 +107,5 @@
         </sensor>
     </gazebo>
-    <!--            Wheels        -->
+    <!--            Car Parts           -->
     <!-- Left front wheel -->
     <gazebo reference="LEFT_FRONT_WHEEL">

Commit message: Teleop twist keyboard functioning

File: ars_description/urdf/arc.xacro (robot description, xacro)
@@ -10,6 +10,6 @@
     <xacro:include filename="$(find ars_description)/urdf/sensors/imu.xacro"/>
     <xacro:include filename="$(find ars_description)/urdf/sensors/lidar.xacro"/>
+    <!--<xacro:include filename="$(find ars_description)/urdf/transmissions.xacro"/>-->
     <xacro:include filename="$(find ars_description)/urdf/gazebo.xacro"/>
-    <xacro:include filename="$(find ars_description)/urdf/transmissions.xacro"/>
     <xacro:chassis/>
     <xacro:hinge prefix="LEFT"

File: ars_description/urdf/gazebo.xacro (robot description, xacro)
@@ -5,51 +5,21 @@
             <plugin>ign_ros2_control/IgnitionSystem</plugin>
         </hardware>
-        <joint name="LEFT_FRONT_WHEEL_JOINT">
-            <command_interface name="velocity">
-                <param name="min">-1000</param>
-                <param name="max">1000</param>
-            </command_interface>
+        <joint name="LEFT_HINGE_JOINT">
+            <command_interface name="position"/>
             <state_interface name="position"/>
-            <state_interface name="velocity"/>
-        </joint>
-        <joint name="RIGHT_FRONT_WHEEL_JOINT">
-            <command_interface name="velocity">
-                <param name="min">-1000</param>
-                <param name="max">1000</param>
-            </command_interface>
-            <state_interface name="position"/>
-            <state_interface name="velocity"/>
-        </joint>
-        <joint name="LEFT_HINGE_JOINT">
-            <command_interface name="velocity">
-                <param name="min">-1000</param>
-                <param name="max">1000</param>
-            </command_interface>
-            <state_interface name="position"/>
-            <state_interface name="velocity"/>
         </joint>
         <joint name="RIGHT_HINGE_JOINT">
-            <command_interface name="velocity">
-                <param name="min">-1000</param>
-                <param name="max">1000</param>
-            </command_interface>
+            <command_interface name="position"/>
             <state_interface name="position"/>
-            <state_interface name="velocity"/>
         </joint>
         <joint name="LEFT_REAR_WHEEL_JOINT">
-            <command_interface name="velocity">
-                <param name="min">-1000</param>
-                <param name="max">1000</param>
-            </command_interface>
+            <command_interface name="velocity"/>
+            <state_interface name="velocity"/>
             <state_interface name="position"/>
-            <state_interface name="velocity"/>
         </joint>
         <joint name="RIGHT_REAR_WHEEL_JOINT">
-            <command_interface name="velocity">
-                <param name="min">-1000</param>
-                <param name="max">1000</param>
-            </command_interface>
+            <command_interface name="velocity"/>
+            <state_interface name="velocity"/>
             <state_interface name="position"/>
-            <state_interface name="velocity"/>
         </joint>
     </ros2_control>
@@ -122,66 +92,3 @@
         <preserveFixedJoint>true</preserveFixedJoint>
     </gazebo>
-    <!--            Car Parts           -->
-    <!-- Left front wheel -->
-    <gazebo reference="LEFT_FRONT_WHEEL">
-        <mu1 value="${friction_coeff}"/>
-        <mu2 value="${friction_coeff}"/>
-        <fdir1 value="1 0 0"/>
-        <kp>10000000.0</kp>
-        <kd>1.0</kd>
-        <minDepth>0.005</minDepth>
-        <maxVel>100.0</maxVel>
-        <material>Gazebo/DarkGrey</material>
-    </gazebo>
-    <!-- Right front wheel -->
-    <gazebo reference="RIGHT_FRONT_WHEEL">
-        <mu1 value="${friction_coeff}"/>
-        <mu2 value="${friction_coeff}"/>
-        <fdir1 value="1 0 0"/>
-        <kp>10000000.0</kp>
-        <kd>1.0</kd>
-        <minDepth>0.005</minDepth>
-        <maxVel>100.0</maxVel>
-        <material>Gazebo/DarkGrey</material>
-    </gazebo>
-    <!-- Left rear wheel -->
-    <gazebo reference="LEFT_REAR_WHEEL">
-        <mu1 value="${friction_coeff}"/>
-        <mu2 value="${friction_coeff}"/>
-        <fdir1 value="1 0 0"/>
-        <kp>10000000.0</kp>
-        <kd>1.0</kd>
-        <minDepth>0.005</minDepth>
-        <maxVel>100.0</maxVel>
-        <material>Gazebo/DarkGrey</material>
-    </gazebo>
-    <!-- Right rear wheel -->
-    <gazebo reference="RIGHT_REAR_WHEEL">
-        <mu1 value="${friction_coeff}"/>
-        <mu2 value="${friction_coeff}"/>
-        <fdir1 value="1 0 0"/>
-        <kp>10000000.0</kp>
-        <kd>1.0</kd>
-        <minDepth>0.005</minDepth>
-        <maxVel>100.0</maxVel>
-        <material>Gazebo/DarkGrey</material>
-    </gazebo>
-    <!-- Left hinge -->
-    <gazebo reference="LEFT_WHEEL_HINGE">
-        <mu1 value="0.0"/>
-        <mu2 value="0.0"/>
-        <kp>10000000.0</kp>
-        <kd>1.0</kd>
-        <fdir1 value="0 1 0"/>
-        <material>Gazebo/DarkGrey</material>
-    </gazebo>
-    <!-- Right hinge -->
-    <gazebo reference="RIGHT_WHEEL_HINGE">
-        <mu1 value="0.0"/>
-        <mu2 value="0.0"/>
-        <kp>10000000.0</kp>
-        <kd>1.0</kd>
-        <fdir1 value="0 1 0"/>
-        <material>Gazebo/DarkGrey</material>
-    </gazebo>
 </robot>

File: ars_description/urdf/parts/hinge.xacro (robot description, xacro)
@@ -8,5 +8,5 @@
             <axis xyz="0 -1 0" rpy="0 0 0"/>
             <dynamics damping="0.0" friction="0.0"/>
-            <limit lower="-0.53" upper="0.53" effort="100" velocity="1"/>
+            <limit lower="-0.53" upper="0.53" effort="100.0" velocity="5.0"/>
         </joint>
         <link name="${prefix}_HINGE">

Commit message: base_link to ground

File: ars_description/urdf/arc.xacro (robot description, xacro)
@@ -10,5 +10,4 @@
     <xacro:include filename="$(find ars_description)/urdf/sensors/imu.xacro"/>
     <xacro:include filename="$(find ars_description)/urdf/sensors/lidar.xacro"/>
-    <!--<xacro:include filename="$(find ars_description)/urdf/transmissions.xacro"/>-->
     <xacro:include filename="$(find ars_description)/urdf/ros2_control.xacro"/>
     <xacro:chassis/>

File: ars_description/urdf/parts/chassis.xacro (robot description, xacro)
@@ -34,5 +34,5 @@
             <parent link="base_link"/>
             <child link="chassis"/>
-            <origin xyz="0 0 0" rpy="0 0 0"/>
+            <origin xyz="0 0 ${wheelRadius - wheelHeight + chassisHeight/2.0}" rpy="0 0 0"/>
         </joint>
     </xacro:macro>

File: ars_description/urdf/parts/hinge.xacro (robot description, xacro)
@@ -3,5 +3,5 @@
     <xacro:macro name="hinge" params="prefix X Y">
         <joint name="${prefix}_HINGE_JOINT" type="continuous">
-            <parent link="${base_link_name}"/>
+            <parent link="chassis"/>
             <child link="${prefix}_HINGE"/>
             <origin xyz="${X} ${Y} ${wheelHeight - chassisHeight/2.0}" rpy="-${0.5*PI} 0.0 0.0"/>

File: ars_description/urdf/parts/rear_wheel.xacro (robot description, xacro)
@@ -3,5 +3,5 @@
     <xacro:macro name="rear_wheel" params="prefix X Y friction_coeff:=0.7 transmission_reduction:=1" >
         <joint name="${prefix}_REAR_WHEEL_JOINT" type="continuous">
-            <parent link="${base_link_name}"/>
+            <parent link="chassis"/>
             <child link="${prefix}_REAR_WHEEL"/>
             <origin xyz="${X} ${Y} ${wheelHeight - chassisHeight/2.0}" rpy="${PI/2} 0 0" />

File: ars_description/urdf/sensors/imu.xacro (robot description, xacro)
@@ -5,5 +5,5 @@
         <joint name="imu_joint" type="fixed">
             <origin xyz="${imu_origin_xyz}" rpy="${imu_origin_rpy}"/>
-            <parent link="${base_link}"/>
+            <parent link="chassis"/>
             <child link="imu_link"/>
         </joint>

File: ars_description/urdf/sensors/lidar.xacro (robot description, xacro)
@@ -5,5 +5,5 @@
         <joint name="lidar_joint" type="fixed">
             <origin xyz="${lidar_origin_xyz}" rpy="${lidar_origin_rpy}"/>
-            <parent link="${base_link}"/>
+            <parent link="chassis"/>
             <child link="lidar_link"/>
         </joint>
