Commit message: No transform between odom and base_link

File: ars_description/urdf/arc.urdf (robot description, URDF)
Before this commit: robot arc, 10 links, 9 joints
Joints:
- joint LEFT_HINGE_JOINT: limit lower=-0.53 upper=0.53 effort=100 velocity=1 -> lower=-0.53 upper=0.53 effort=100.0 velocity=5.0
- joint RIGHT_HINGE_JOINT: limit lower=-0.53 upper=0.53 effort=100 velocity=1 -> lower=-0.53 upper=0.53 effort=100.0 velocity=5.0

File: ars_description/urdf/arc.xacro (robot description, xacro)
@@ -11,5 +11,5 @@
     <xacro:include filename="$(find ars_description)/urdf/sensors/lidar.xacro"/>
     <!--<xacro:include filename="$(find ars_description)/urdf/transmissions.xacro"/>-->
-    <xacro:include filename="$(find ars_description)/urdf/gazebo.xacro"/>
+    <xacro:include filename="$(find ars_description)/urdf/ros2_control.xacro"/>
     <xacro:chassis/>
     <xacro:hinge prefix="LEFT"

File: ars_description/urdf/parts/front_wheel.xacro (robot description, xacro)
@@ -7,7 +7,5 @@
             <origin xyz="0 0 ${Y}" rpy="0 0 0" />
             <axis xyz="0 0 1" rpy="0 0 0" />
-            <dynamics damping="0.0" friction="0.0"/>
-            <limit effort="100" velocity="200"/>
-            <joint_properties damping="0.2" friction="0.2"/>
+            <dynamics damping="0.2"/>
         </joint>
         <link name="${prefix}_FRONT_WHEEL">

File: ars_description/urdf/parts/hinge.xacro (robot description, xacro)
@@ -2,11 +2,9 @@
 <robot xmlns:xacro="http://www.ros.org/wiki/xacro">
     <xacro:macro name="hinge" params="prefix X Y">
-        <joint name="${prefix}_HINGE_JOINT" type="revolute">
+        <joint name="${prefix}_HINGE_JOINT" type="continuous">
             <parent link="${base_link_name}"/>
             <child link="${prefix}_HINGE"/>
             <origin xyz="${X} ${Y} ${wheelHeight - chassisHeight/2.0}" rpy="-${0.5*PI} 0.0 0.0"/>
             <axis xyz="0 -1 0" rpy="0 0 0"/>
-            <dynamics damping="0.0" friction="0.0"/>
-            <limit lower="-0.53" upper="0.53" effort="100.0" velocity="5.0"/>
         </joint>
         <link name="${prefix}_HINGE">

File: ars_description/urdf/parts/rear_wheel.xacro (robot description, xacro)
@@ -7,7 +7,4 @@
             <origin xyz="${X} ${Y} ${wheelHeight - chassisHeight/2.0}" rpy="${PI/2} 0 0" />
             <axis xyz="0 0 -1" rpy="0 0 0" />
-            <dynamics damping="0.0" friction="0.0"/>
-            <limit effort="100" velocity="200"/>
-            <joint_properties damping="0.2" friction="0.2"/>
         </joint>
         <link name="${prefix}_REAR_WHEEL">

File: ars_description/urdf/sensors/imu.xacro (robot description, xacro)
@@ -28,4 +28,16 @@
             </collision>
         </link>
+        <gazebo reference="imu_link">
+            <sensor name="imu_sensor" type="imu">
+                <always_on>1</always_on>
+                <update_rate>${imu_update_rate}</update_rate>
+                <ignition_frame_id>imu_link</ignition_frame_id>
+                <visualize>true</visualize>
+                <topic>${imu_topic}</topic>
+            </sensor>
+        </gazebo>
+        <gazebo reference="imu_joint">
+            <preserveFixedJoint>true</preserveFixedJoint>
+        </gazebo>
     </xacro:macro>
 </robot>

File: ars_description/urdf/sensors/lidar.xacro (robot description, xacro)
@@ -28,4 +28,42 @@
             </collision>
         </link>
+        <gazebo reference="lidar_link">
+            <sensor name='gpu_lidar' type='gpu_lidar'>
+                <topic>${lidar_topic}</topic>
+                <update_rate>${lidar_update_rate}</update_rate>
+                <alwaysOn>1</alwaysOn>
+                <visualize>true</visualize>
+                <ignition_frame_id>lidar_link</ignition_frame_id>
+                <lidar>
+                    <scan>
+                        <horizontal>
+                            <samples>640</samples>
+                            <resolution>1</resolution>
+                            <min_angle>-1.396263</min_angle>
+                            <max_angle>1.396263</max_angle>
+                        </horizontal>
+                        <vertical>
+                        <samples>1</samples>
+                        <resolution>1</resolution>
+                        <min_angle>0.0</min_angle>
+                        <max_angle>0.0</max_angle>
+                        </vertical>
+                    </scan>
+                    <range>
+                        <min>0.08</min>
+                        <max>10</max>
+                        <resolution>0.01</resolution>
+                    </range>
+                    <noise>
+                        <type>gaussian</type>
+                        <mean>0.0</mean>
+                        <stddev>0.001</stddev>
+                    </noise>
+                </lidar>
+            </sensor>
+        </gazebo>
+        <gazebo reference="lidar_joint">
+            <preserveFixedJoint>true</preserveFixedJoint>
+        </gazebo>
     </xacro:macro>
 </robot>

Commit message: Robot still turns diff drive like in RViz

File: ars_description/urdf/arc.urdf (robot description, URDF)
Before this commit: robot arc, 10 links, 9 joints
Links:
- removed link base_inertia
- added link chassis, mass 2.3; collision box size=0.57 0.29 0.075; visual box size=0.57 0.29 0.075
- link LEFT_FRONT_WHEEL: geometry collision sphere radius=0.055; visual cylinder length=0.037 radius=0.055
- link LEFT_REAR_WHEEL: geometry collision sphere radius=0.055; visual cylinder length=0.037 radius=0.055
- link RIGHT_FRONT_WHEEL: geometry collision sphere radius=0.055; visual cylinder length=0.037 radius=0.055
- link RIGHT_REAR_WHEEL: geometry collision sphere radius=0.055; visual cylinder length=0.037 radius=0.055
- link base_link: geometry 
Joints:
- removed joint base_to_base_inertia
- added joint chassis_joinz: type fixed, parent base_link, child chassis, origin xyz=0 0 0.08449999999999999 rpy=0 0 0
- joint LEFT_FRONT_WHEEL_JOINT: limit effort=100 velocity=200 -> (none)
- joint LEFT_HINGE_JOINT: limit lower=-0.53 upper=0.53 effort=100.0 velocity=5.0 -> (none); parent base_link -> chassis; type revolute -> continuous
- joint LEFT_REAR_WHEEL_JOINT: limit effort=100 velocity=200 -> (none); origin xyz=-0.162 0.1735 -0.0295 rpy=1.5707963267948966 0 0 -> xyz=-0.162 0.19349999999999998 -0.0295 rpy=1.5707963267948966 0 0; parent base_link -> chassis
- joint RIGHT_FRONT_WHEEL_JOINT: limit effort=100 velocity=200 -> (none)
- joint RIGHT_HINGE_JOINT: limit lower=-0.53 upper=0.53 effort=100.0 velocity=5.0 -> (none); parent base_link -> chassis; type revolute -> continuous
- joint RIGHT_REAR_WHEEL_JOINT: limit effort=100 velocity=200 -> (none); origin xyz=-0.162 -0.1735 -0.0295 rpy=1.5707963267948966 0 0 -> xyz=-0.162 -0.19349999999999998 -0.0295 rpy=1.5707963267948966 0 0; parent base_link -> chassis
- joint imu_joint: parent base_link -> chassis
- joint lidar_joint: parent base_link -> chassis

Commit message: Preparing for class. LiDAR doesn't work properly.

File: ars_description/urdf/arc.urdf (robot description, URDF)
Before this commit: robot arc, 10 links, 9 joints
Joints:
- joint LEFT_HINGE_JOINT: axis 0 -1 0 -> 0 1 0
- joint RIGHT_HINGE_JOINT: axis 0 -1 0 -> 0 1 0

File: ars_description/urdf/properties.xacro (robot description, xacro)
@@ -28,5 +28,5 @@
     <xacro:property name="lidar_radius"		value="0.0516"/>
     <xacro:property name="lidar_mass"		value="0.15"/>
-    <xacro:property name="lidar_update_rate"		value="400"/>
+    <xacro:property name="lidar_update_rate"		value="20"/>
     <xacro:property name="lidar_topic" 			value="/scan"/>
     <!-- IMU properties -->

File: ars_description/urdf/sensors/lidar.xacro (robot description, xacro)
@@ -44,13 +44,13 @@
                         </horizontal>
                         <vertical>
-                        <samples>1</samples>
-                        <resolution>1</resolution>
-                        <min_angle>0.0</min_angle>
-                        <max_angle>0.0</max_angle>
+                            <samples>1</samples>
+                            <resolution>1</resolution>
+                            <min_angle>0.0</min_angle>
+                            <max_angle>0.0</max_angle>
                         </vertical>
                     </scan>
                     <range>
-                        <min>0.08</min>
-                        <max>10</max>
+                        <min>0.5</min>
+                        <max>500</max>
                         <resolution>0.01</resolution>
                     </range>
@@ -60,4 +60,5 @@
                         <stddev>0.001</stddev>
                     </noise>
+                    <visibility_mask>4294967294</visibility_mask>
                 </lidar>
             </sensor>
